Commit message: Add KR240-R3330 Meshes

File: kuka_fortec_support/urdf/kr240_r3330_macro.xacro (robot description, xacro)
@@ -114,5 +114,5 @@
       <child link="${prefix}link_1"/>
       <limit effort="15000.0E0" lower="${radians(-185)}" upper="${radians(185)}" velocity="${radians(100)}"/>
-      <origin rpy="-3.141592653589793 0.0 -0.0" xyz="0.0 0.0 0.0"/>
+      <origin rpy="-3.141592653589793 0.0 0.0" xyz="0.0 0.0 1.045"/>
       <parent link="${prefix}base_link"/>
     </joint>
@@ -121,5 +121,5 @@
       <child link="${prefix}link_2"/>
       <limit effort="17880.0E0" lower="${radians(-130)}" upper="${radians(20)}" velocity="${radians(90)}"/>
-      <origin rpy="${pi/2.0} 0.0 -0.0" xyz="0.5 0.0 -1.045"/>
+      <origin rpy="${pi/2.0} 0.0 -0.0" xyz="0.5 0.0 0"/>
       <parent link="${prefix}link_1"/>
     </joint>
@@ -149,5 +149,5 @@
       <child link="${prefix}link_6"/>
       <limit effort="2675.4449432041E0" lower="${radians(-350)}" upper="${radians(350)}" velocity="${radians(160)}"/>
-      <origin rpy="${pi/2.0} 0.0 -0.0" xyz="0.0 0.0 0.0"/>
+      <origin rpy="${pi/2.0} 0.0 -0.0" xyz="0.0 0.29 0.0"/>
       <parent link="${prefix}link_5"/>
     </joint>
@@ -163,5 +163,5 @@
     <joint name="${prefix}link6-flange" type="fixed">
       <child link="${prefix}flange"/>
-      <origin rpy="0 ${pi/2} -0.0" xyz="0.0 0.0 -0.29"/>
+      <origin rpy="0 ${pi/2} -0.0" xyz="0.0 0.0 0.0"/>
       <parent link="${prefix}link_6"/>
     </joint>
@@ -170,5 +170,5 @@
     <joint name="${prefix}link6-tool0" type="fixed">
       <child link="${prefix}tool0"/>
-      <origin rpy="0 ${pi} -0.0" xyz="0.0 0.0 -0.29"/>
+      <origin rpy="0 ${pi} -0.0" xyz="0.0 0.0 0.0"/>
       <parent link="${prefix}link_6"/>
     </joint>
